File: arduino/bridge/bridge.kicad_pcb (KiCad board)
At the start: 2 copper layers, 3 parts, among them J1 Conn_01x15_Socket, J2 Conn_01x15_Socket, J3 Conn_01x08_Socket

Commit message: epochTime and bridge update
Routing:
- net Rot: track 140.1 -> 134.8 mm
- net Rot/RST: track 81.1 -> 79.9 mm
Changed lines of the file:
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@@
   (segment (start 51 63) (end 48.905 60.905) (width 0.25) (layer "F.Cu") (net 10))
   (segment (start 60 114.65) (end 52.65 114.65) (width 0.25) (layer "F.Cu") (net 10))
+  (segment (start 41 60) (end 41 63) (width 0.25) (layer "F.Cu") (net 13))
+  (segment (start 48 116) (end 51.73 119.73) (width 0.25) (layer "F.Cu") (net 13))
+  (segment (start 51.73 119.73) (end 60 119.73) (width 0.25) (layer "F.Cu") (net 13))
+  (segment (start 43 65) (end 46 65) (width 0.25) (layer "F.Cu") (net 13))
+  (segment (start 46 65) (end 48 67) (width 0.25) (layer "F.Cu") (net 13))
   (segment (start 41 63) (end 43 65) (width 0.25) (layer "F.Cu") (net 13))
-  (segment (start 46 65) (end 48 67) (width 0.25) (layer "F.Cu") (net 13))
-  (segment (start 49.73 119.73) (end 60 119.73) (width 0.25) (layer "F.Cu") (net 13))
-  (segment (start 48 67) (end 48 118) (width 0.25) (layer "F.Cu") (net 13))
+  (segment (start 48 67) (end 48 116) (width 0.25) (layer "F.Cu") (net 13))
+  (segment (start 46 58.365) (end 42.635 58.365) (width 0.25) (layer "F.Cu") (net 13))
   (segment (start 42.635 58.365) (end 41 60) (width 0.25) (layer "F.Cu") (net 13))
-  (segment (start 43 65) (end 46 65) (width 0.25) (layer "F.Cu") (net 13))
-  (segment (start 46 58.365) (end 42.635 58.365) (width 0.25) (layer "F.Cu") (net 13))
-  (segment (start 48 118) (end 49.73 119.73) (width 0.25) (layer "F.Cu") (net 13))
-  (segment (start 41 60) (end 41 63) (width 0.25) (layer "F.Cu") (net 13))
   (segment (start 80.625 43.125) (end 83 45.5) (width 0.25) (layer "F.Cu") (net 18))
   (segment (start 83 93) (end 84.33 94.33) (width 0.25) (layer "F.Cu") (net 18))
@@
   (segment (start 80 48) (end 77.665 45.665) (width 0.25) (layer "F.Cu") (net 22))
   (segment (start 77.665 45.665) (end 46 45.665) (width 0.25) (layer "F.Cu") (net 22))
-  (segment (start 41 49) (end 42.745 50.745) (width 0.25) (layer "F.Cu") (net 23))
-  (segment (start 94 108) (end 94 43) (width 0.25) (layer "F.Cu") (net 23))
-  (segment (start 94 43) (end 91 40) (width 0.25) (layer "F.Cu") (net 23))
-  (segment (start 88 109.57) (end 92.43 109.57) (width 0.25) (layer "F.Cu") (net 23))
+  (segment (start 42.745 50.745) (end 41 49) (width 0.25) (layer "F.Cu") (net 23))
+  (segment (start 94 108) (end 92.43 109.57) (width 0.25) (layer "F.Cu") (net 23))
+  (segment (start 41 49) (end 41 42) (width 0.25) (layer "F.Cu") (net 23))
+  (segment (start 92.43 109.57) (end 88 109.57) (width 0.25) (layer "F.Cu") (net 23))
+  (segment (start 85.5 79.5) (end 94 88) (width 0.25) (layer "F.Cu") (net 23))
+  (segment (start 41 42) (end 43 40) (width 0.25) (layer "F.Cu") (net 23))
+  (segment (start 43 40) (end 82 40) (width 0.25) (layer "F.Cu") (net 23))
   (segment (start 87.57 110) (end 88 109.57) (width 0.25) (layer "F.Cu") (net 23))
-  (segment (start 91 40) (end 43 40) (width 0.25) (layer "F.Cu") (net 23))
-  (segment (start 42.745 50.745) (end 46 50.745) (width 0.25) (layer "F.Cu") (net 23))
-  (segment (start 92.43 109.57) (end 94 108) (width 0.25) (layer "F.Cu") (net 23))
-  (segment (start 41 42) (end 41 49) (width 0.25) (layer "F.Cu") (net 23))
-  (segment (start 43 40) (end 41 42) (width 0.25) (layer "F.Cu") (net 23))
+  (segment (start 46 50.745) (end 42.745 50.745) (width 0.25) (layer "F.Cu") (net 23))
+  (segment (start 94 88) (end 94 108) (width 0.25) (layer "F.Cu") (net 23))
+  (segment (start 82 40) (end 85.5 43.5) (width 0.25) (layer "F.Cu") (net 23))
+  (segment (start 85.5 43.5) (end 85.5 79.5) (width 0.25) (layer "F.Cu") (net 23))
   (segment (start 77 51) (end 74.205 48.205) (width 0.25) (layer "F.Cu") (net 24))
   (segment (start 77 110) (end 77 51) (width 0.25) (layer "F.Cu") (net 24))
